Commit message: New updates on the robot code and simulation

File: deps/BipedRobot/biped_robot.urdf (robot description, URDF)
Before this commit: robot biped_robot, 6 links, 5 joints
Links:
- added link l_foot_link, mass 1; visual sphere radius=.03
- added link r_foot_link, mass 1; visual sphere radius=.03
Joints:
- added joint l_foot_joint: type fixed, parent l_leg_link, child l_foot_link, origin xyz=0 0 -1
- added joint r_foot_joint: type fixed, parent r_leg_link, child r_foot_link, origin xyz=0 0 -1
